File: project/project.kicad_pcb (KiCad board)
At the start: 2 copper layers, 8.6 x 4.6 mm, 67 parts, among them J1 Conn_02x16_Odd_Even, J2 TYPE-C 6P(040新), J3 Conn_01x02_Pin, SW1 SS-12D10L9, U1 DRV8833PWPR, U10 TPS22965DSGR, U11 TS5A3159ADBVR, U2 CH224K, U3 DRV8833PWPR, U4 AP63203WU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

Commit message: Routing
Parts:
- added JP1: Jumper_2_Open, Jumper:SolderJumper-2_P1.3mm_Open_RoundedPad1.0x1.5mm, F.Cu at (122.8, 81.9)
- added JP2: Jumper_2_Open, Jumper:SolderJumper-2_P1.3mm_Open_RoundedPad1.0x1.5mm, F.Cu at (161.7, 98.0)
- added JP3: Jumper_2_Open, Jumper:SolderJumper-2_P1.3mm_Open_RoundedPad1.0x1.5mm, F.Cu at (122.8, 85.5)
- added JP4: Jumper_2_Open, Jumper:SolderJumper-2_P1.3mm_Open_RoundedPad1.0x1.5mm, F.Cu at (122.8, 89.0)
- J2: footprint Library:CONN_TYPE-C-6P_SHN -> Connector_USB:USB_C_Receptacle_GCT_USB4135-GF-A_6P_TopMnt_Horizontal
- R16: value 1m -> 0.5m; footprint Resistor_SMD:R_0402_1005Metric_Pad0.72x0.64mm_HandSolder -> Resistor_THT:R_Axial_Shunt_L22.2mm_W8.0mm_PS14.30mm_P25.40mm
- moved TP12 28.3 mm to (99.5, 77.5)
- moved TP8 20.6 mm to (124.0, 99.5)
- moved TP7 11.4 mm to (105.0, 102.5)
- moved TP9 10.5 mm to (99.5, 94.0)
- moved TP13 8.73 mm to (101.5, 73.5)
- moved U3 4.61 mm to (107.6, 95.3)
- moved TP10 4.50 mm to (98.0, 66.0)
- moved TP6 4.03 mm to (99.0, 89.0)
- moved TP11 4.00 mm to (97.0, 72.5)
- moved SW1 2.92 mm to (156.0, 81.0)
Connections:
- C10 pad 1: Net-(U4-FB) -> Net-(JP2-B)
- L1 pad 2: Net-(U4-FB) -> Net-(JP2-B)
- TP5 pad 1: Net-(U4-FB) -> Net-(JP2-B)
- U2 pad 5: Net-(U2-DM) -> Net-(JP4-B)
- U4 pad 1: Net-(U4-FB) -> Net-(JP2-B)
- U5 pad 4: Net-(U4-FB) -> Net-(JP2-B)
- U5 pad 8: Net-(U4-FB) -> Net-(JP2-B)
Routing:
- net GND: track 0.00 -> 412.8 mm, vias 0 -> 8
- net /Battery: track 0.00 -> 265.0 mm, vias 0 -> 15
- net Net-(JP2-B): track 0.00 -> 130.7 mm, vias 0 -> 6
- net /5V Out: track 0.00 -> 104.3 mm, vias 0 -> 4
- net /BATT: track 0.00 -> 95.0 mm, vias 0 -> 3
- net /MOTOR2_A_OUT: track 0.00 -> 94.1 mm, vias 0 -> 6
- net /MOTOR4_A_OUT: track 0.00 -> 88.8 mm, vias 0 -> 3
- net /EXT_LOAD1_OUT: track 0.00 -> 85.6 mm, vias 0 -> 3
- net /EXT_LOAD2_OUT: track 0.00 -> 82.2 mm, vias 0 -> 4
- net /MOTOR2_CTRL2: track 0.00 -> 81.5 mm, vias 0 -> 1
- net /MOTOR2_CTRL1: track 0.00 -> 78.7 mm, vias 0 -> 2
- net /3V3 Out: track 0.00 -> 73.5 mm, vias 0 -> 7
- net Net-(U2-VBUS): track 0.00 -> 70.5 mm, vias 0 -> 2
- net /I2C1_SCL: track 0.00 -> 69.8 mm, vias 0 -> 3
- net /Motor2_A_OUT: track 0.00 -> 67.6 mm
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- added copper zone on F.Cu, net (none)
Other:
- board outline removed
