File: project/project.kicad_pcb (KiCad board)
At the start: 2 copper layers, 67 parts, among them J1 Conn_02x16_Odd_Even, J2 TYPE-C 6P(040新), J3 Conn_01x02_Pin, SW1 SS-12D10L9, U1 DRV8833PWPR, U10 TPS22965DSGR, U11 TS5A3159ADBVR, U2 CH224K, U3 DRV8833PWPR, U4 AP63203WU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

Commit message: checks
Parts:
- R16: footprint Resistor_THT:R_Axial_Shunt_L22.2mm_W8.0mm_PS14.30mm_P25.40mm -> Resistor_SMD:R_Shunt_Vishay_WSR2_WSR3
- moved R16 14.4 mm to (160.0, 90.0)
Routing:
- net /MOTOR4_B_OUT: track 87.1 -> 139.4 mm, vias 3 -> 6
- net /Motor4_A_OUT: track 65.3 -> 99.6 mm
- net /Motor4_B_OUT: track 92.0 -> 123.5 mm, vias 2 -> 5
- net Net-(U8-IN+): track 34.7 -> 50.5 mm
- net /BATT: track 94.4 -> 101.2 mm
- net /Battery: track 295.6 -> 297.0 mm, vias 7 -> 8
- net Net-(J2-VBUS-PadA9): track 26.4 -> 27.1 mm
- net Net-(U6-ADJ): track 44.5 -> 45.0 mm
- net /MOTOR4_A_OUT: vias 4 -> 5

Commit message: Updates
Changes datasheet names,updates PCB,fixex errors
Parts:
- J3: footprint Connector_PinHeader_2.00mm:PinHeader_1x02_P2.00mm_Vertical -> Connector_JST:JST_PH_B2B-PH-K_1x02_P2.00mm_Vertical
- moved U10 81.2 mm to (185.5, 98.8), turned to 0 degrees
- moved C17 72.6 mm to (181.0, 99.1), turned to -90 degrees
- moved SW1 71.9 mm to (185.0, 61.5)
- moved J3 71.6 mm to (183.0, 89.0), turned to 0 degrees
- moved JP3 61.6 mm to (189.7, 71.5), turned to 0 degrees
- moved L2 61.3 mm to (149.7, 58.0), turned to 0 degrees
- moved JP2 61.2 mm to (190.7, 78.5), turned to 0 degrees
- moved TP5 61.0 mm to (177.3, 65.5), turned to 0 degrees
- moved C13 61.0 mm to (162.7, 55.0), turned to 0 degrees
- moved R2 59.9 mm to (141.3, 67.7)
- moved U2 59.7 mm to (136.8, 58.0), turned to 0 degrees
- moved C16 58.2 mm to (166.5, 91.6), turned to -90 degrees
- moved C6 55.7 mm to (159.2, 54.6)
- moved C15 53.1 mm to (143.2, 64.0), turned to -90 degrees
- moved R10 52.4 mm to (152.7, 62.1), turned to -90 degrees
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Connections:
- J1 pad 1: /Motor2_B_OUT -> /MOTOR2_B_OUT
- J1 pad 2: /Motor2_A_OUT -> /MOTOR2_A_OUT
- J1 pad 3: /Motor4_A_OUT -> /MOTOR4_A_OUT
- J1 pad 5: /Motor4_B_OUT -> /MOTOR4_B_OUT
- R8 pad 1: /3V3 -> /3V3 Out
- R9 pad 1: /3V3 -> /3V3 Out
- U3 pad 10: /MOTOR3_CTRL2 -> /MOTOR4_CTRL2
- U3 pad 9: /MOTOR3_CTRL1 -> /MOTOR4_CTRL1
- U7 pad 6: Net-(U7-OC) -> (no net)
- U8 pad 4: /3V3 -> /3V3 Out
- U8 pad 7: /3V3 -> /3V3 Out
Routing:
- net GND: track 367.5 -> 0.00 mm, vias 5 -> 0
- net /Battery: track 297.0 -> 0.00 mm, vias 8 -> 0
- net /MOTOR4_B_OUT: track 139.4 -> 0.00 mm, vias 6 -> 0
- net /Motor4_B_OUT: track 123.5 -> 0.00 mm, vias 5 -> 0
- net /EXT_LOAD1_OUT: track 107.7 -> 0.00 mm, vias 1 -> 0
- net /5V Out: track 105.8 -> 0.00 mm, vias 7 -> 0
- net /BATT: track 101.2 -> 0.00 mm, vias 3 -> 0
- net /Motor4_A_OUT: track 99.6 -> 0.00 mm, vias 1 -> 0
- net /3V3 Out: track 84.9 -> 0.00 mm, vias 3 -> 0
- net Net-(U8-IN-): track 58.9 -> 0.00 mm, vias 4 -> 0
- net /FAST_CHARGE_CTRL: track 58.6 -> 0.00 mm, vias 1 -> 0
- net /HV: track 53.5 -> 0.00 mm, vias 1 -> 0
- net /MOTOR1_B_OUT: track 53.0 -> 0.00 mm, vias 3 -> 0
- net Net-(U7-FB): track 52.4 -> 0.00 mm, vias 5 -> 0
- net Net-(U8-IN+): track 50.5 -> 0.00 mm, vias 3 -> 0
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- removed copper zone on F.Cu, net (none)
Other:
- board outline added: 80 x 60 mm
- board text removed: "TMBTLA001 MDLOXO001 65"

Commit message: fixing errors on PCB
Parts:
- added R17: 200m, Resistor_SMD:R_0402_1005Metric_Pad0.72x0.64mm_HandSolder, F.Cu at (130.0, 79.0)
- added R18: 200m, Resistor_SMD:R_0402_1005Metric_Pad0.72x0.64mm_HandSolder, F.Cu at (117.5, 97.5)
- moved TP8 21.5 mm to (127.0, 89.5)
- moved TP6 9.55 mm to (131.0, 69.0)
- moved TP7 9.55 mm to (131.0, 74.0)
- moved TP9 9.12 mm to (127.0, 84.0)
- moved TP12 3.81 mm to (118.5, 102.0)
Connections:
- U1 pad 3: GND -> Net-(U1-AISEN)
- U1 pad 6: GND -> Net-(U1-AISEN)
- U3 pad 3: GND -> Net-(U3-AISEN)
- U3 pad 6: GND -> Net-(U3-AISEN)
