File: project/project.kicad_pcb (KiCad board)
At the start: 2 copper layers, 80 x 60 mm, 69 parts, among them J1 Conn_02x16_Odd_Even, J2 TYPE-C 6P(040新), J3 Conn_01x02_Pin, SW1 SS-12D10L9, U1 DRV8833PWPR, U10 TPS22965DSGR, U11 TS5A3159ADBVR, U2 CH224K, U3 DRV8833PWPR, U4 AP63203WU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

Commit message: import/export
Parts:
- removed U11: TS5A3159ADBVR, Package_TO_SOT_SMD:SOT-23-6
- added U12: MT3608L, Footprint:SOT-23-6_L2.9-W1.6-P0.95-LS2.8-BL_3, F.Cu at (136.0, 106.5)
- U1, U3: footprint Footprint:DRV8833PWPR -> Footprint:TSSOP-16_L5.0-W4.4-P0.65-LS6.4-BL-EP
- U10, U9: footprint Footprint:TPS22965DSGR -> Footprint:SOT-23-6_L2.9-W1.6-P0.95-LS2.8-BR
- U7: value MT3608L -> INA219AIDCNR; footprint Package_SON:WSON-6-1EP_2x2mm_P0.65mm_EP1x1.6mm -> Footprint:SOT-23-8_L3.0-W1.7-P0.65-LS2.8-BR
- U8: value INA219AIDCNR -> TS5A3159ADBVR; footprint Footprint:INA219AIDCNR -> Footprint:SOT-23-6_L2.9-W1.6-P0.95-LS2.8-BR
- moved U8 27.3 mm to (172.0, 91.0), turned to 0 degrees
- moved U7 25.0 mm to (143.5, 78.5), turned to 0 degrees
- moved R10 9.53 mm to (144.4, 99.4), turned to 0 degrees
- moved R7 8.92 mm to (149.0, 100.1), turned to 90 degrees
- moved TP5 8.75 mm to (159.0, 101.0)
- moved C15 7.06 mm to (169.5, 106.5)
- moved JP3 5.52 mm to (137.0, 94.5)
- moved L2 4.74 mm to (142.0, 104.0), turned to 90 degrees
- moved C16 4.47 mm to (138.5, 74.1)
- moved R8 4.47 mm to (139.0, 70.3)
- moved R9 4.47 mm to (143.0, 71.3)
- moved L1 3.81 mm to (145.0, 94.8)
- moved R6 3.77 mm to (140.4, 99.5)
- moved D3 3.55 mm to (136.0, 100.1)
- moved C14 3.51 mm to (132.0, 98.5)
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Connections:
- R11 pad 1: Net-(U5-PROG) -> Net-(U8-NO)
- R11 pad 2: Net-(R11-Pad2) -> GND
- R15 pad 1: Net-(U5-PROG) -> GND
- R15 pad 2: Net-(R15-Pad2) -> Net-(U8-NC)
- R16 pad 2: Net-(U8-IN+) -> Net-(U7-IN+)
- R6 pad 2: Net-(U7-FB) -> Net-(U12-FB)
- R7 pad 1: Net-(U7-FB) -> Net-(U12-FB)
- U7 pad 1: /Battery -> Net-(U7-IN+)
- U7 pad 2: (no net) -> Net-(U7-IN-)
- U7 pad 3: Net-(U7-FB) -> GND
- U7 pad 4: /Battery -> /3V3 Out
- U7 pad 5: Net-(D3-A) -> /I2C1_SCL
- U7 pad 6: (no net) -> /I2C1_SDA
- U8 pad 1: Net-(U8-IN+) -> Net-(U8-NO)
- U8 pad 2: Net-(U8-IN-) -> GND
- U8 pad 3: GND -> Net-(U8-NC)
- U8 pad 4: /3V3 Out -> Net-(U5-PROG)
- U8 pad 5: /I2C1_SCL -> /5V Out
- U8 pad 6: /I2C1_SDA -> /FAST_CHARGE_CTRL
Other:
- board text added: "TMBTLA001 MDLOXO001 GROUP 65"
