File: project/project.kicad_sch (KiCad schematic)
At the start: 63 parts, among them J1 Conn_02x16_Odd_Even, J2 TYPE-C 6P(040新), J3 Conn_01x02_Pin, SW1 SS-12D10L9, U1 DRV8833PWPR, U10 TPS22965DSGR, U2 CH224K, U3 DRV8833PWPR, U4 AP63203WU-7, U5 TP4056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

Commit message: update
Parts:
- added TP1, TP14: TestPoint, TestPoint:TestPoint_Pad_D2.0mm, symbol Connector:TestPoint
- C1, C10, C11, C12, C13, C14, C15, C16, C17, C2, C3, C4, C5, C6, C7, C8, C9: footprint (none) -> Capacitor_SMD:C_0402_1005Metric_Pad0.74x0.62mm_HandSolder
- D1, D2: footprint (none) -> LED_SMD:LED_0402_1005Metric_Pad0.77x0.64mm_HandSolder
- L1: footprint (none) -> Inductor_SMD:L_0402_1005Metric_Pad0.77x0.64mm_HandSolder
- R1, R10, R11, R12, R13, R14, R2, R3, R4, R5, R6, R7, R9: footprint (none) -> Resistor_SMD:R_0402_1005Metric_Pad0.72x0.64mm_HandSolder
- R8: value 3.7k -> 4.7k
- TP10, TP11, TP12, TP13, TP4, TP5, TP6, TP7, TP8, TP9: footprint (none) -> TestPoint:TestPoint_Pad_D2.0mm
- U10, U9: LCSC (none) -> C122837
- U3: LCSC (none) -> C50506
- U8: LCSC (none) -> C87469
Connections:
- net BATT- is gone; now on net GND: U8.2 (IN-)
- net BATT: no longer U8.1 (IN+)
- net BATTERY: now also U8.1 (IN+)
- net CTRL_EXT_LOAD1: no longer U9.3 (ON)
- net CTRL_EXT_LOAD2: now also U9.3 (ON)
- net EXT_LOAD1_OUT: now also TP1.1; no longer R5.1, U9.7 (VOUT), U9.8 (VOUT)
- net EXT_LOAD2_OUT: now also R5.1, U9.7 (VOUT), U9.8 (VOUT), TP14.1
Other:
- note added: "Battery Monitor"

Commit message: update
Parts:
- removed U4: AP63203WU-7, AP63203WU-7_DIO, symbol AP63203WU-7:AP63203WU-7
- added U4: AP63203WU, Package_TO_SOT_SMD:TSOT-23-6, symbol Regulator_Switching:AP63203WU
Connections:
- net 9V: now also U4.2 (EN), U4.3 (IN)
- net GND: now also U4.4 (GND)
- net at C10.1, D1.2 (A), D2.2 (A)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: now also U4.1 (FB)
- net at C9.2, L1.1: now also U4.5 (SW)
- net at C9.1: now also U4.6 (BST)
Changed lines of the file:
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@@
 	)
 	(junction
-		(at 143.51 92.71)
-		(diameter 0)
-		(color 0 0 0 0)
-	)
-	(junction
 		(at 68.58 88.9)
 		(diameter 0)
@@
 	)
 	(junction
+		(at 143.51 92.71)
+		(diameter 0)
+		(color 0 0 0 0)
+	)
+	(junction
 		(at 283.21 31.75)
 		(diameter 0)
@@
 	)
 	(junction
+		(at 104.14 101.6)
+		(diameter 0)
+		(color 0 0 0 0)
+	)
+	(junction
 		(at 149.86 101.6)
 		(diameter 0)
@@
 	(wire
 		(pts
+			(xy 130.81 99.06) (xy 130.81 102.87)
+		)
+		(stroke
+			(width 0)
+			(type default)
+		)
+	)
+	(wire
+		(pts
 			(xy 66.04 96.52) (xy 66.04 118.11)
 		)
@@
 	(wire
 		(pts
+			(xy 127 99.06) (xy 130.81 99.06)
+		)
+		(stroke
+			(width 0)
+			(type default)
+		)
+	)
+	(wire
+		(pts
 			(xy 251.46 31.75) (xy 261.62 31.75)
 		)
@@
 	(wire
 		(pts
+			(xy 137.16 109.22) (xy 116.84 109.22)
+		)
+		(stroke
+			(width 0)
+			(type default)
+		)
+	)
+	(wire
+		(pts
 			(xy 97.79 135.89) (xy 97.79 147.32)
 		)
@@
 	(wire
 		(pts
+			(xy 133.35 99.06) (xy 137.16 99.06)
+		)
+		(stroke
+			(width 0)
+			(type default)
+		)
+	)
+	(wire
+		(pts
 			(xy 100.33 147.32) (xy 100.33 148.59)
 		)
@@
 	(wire
 		(pts
-			(xy 96.52 92.71) (xy 96.52 99.06)
+			(xy 96.52 101.6) (xy 104.14 101.6)
+		)
+		(stroke
+			(width 0)
+			(type default)
+		)
+	)
+	(wire
+		(pts
+			(xy 137.16 102.87) (xy 137.16 101.6)
 		)
 		(stroke
@@
 	(wire
 		(pts
+			(xy 129.54 104.14) (xy 129.54 92.71)
+		)
+		(stroke
+			(width 0)
+			(type default)
+		)
+	)
+	(wire
+		(pts
 			(xy 203.2 78.74) (xy 199.39 78.74)
 		)
@@
 	(wire
 		(pts
+			(xy 104.14 104.14) (xy 106.68 104.14)
+		)
+		(stroke
+			(width 0)
+			(type default)
+		)
+	)
+	(wire
+		(pts
 			(xy 163.83 149.86) (xy 163.83 151.13)
 		)
@@
 	(wire
 		(pts
+			(xy 137.16 104.14) (xy 137.16 109.22)
+		)
+		(stroke
+			(width 0)
+			(type default)
+		)
+	)
+	(wire
+		(pts
+			(xy 104.14 99.06) (xy 106.68 99.06)
+		)
+		(stroke
+			(width 0)
+			(type default)
+		)
+	)
+	(wire
+		(pts
 			(xy 194.31 104.14) (xy 203.2 104.14)
 		)
@@
 	(wire
 		(pts
+			(xy 130.81 102.87) (xy 137.16 102.87)
+		)
+		(stroke
+			(width 0)
+			(type default)
+		)
+	)
+	(wire
+		(pts
 			(xy 134.62 24.13) (xy 152.4 24.13)
 		)
@@
 	(wire
 		(pts
+			(xy 104.14 101.6) (xy 104.14 99.06)
+		)
+		(stroke
+			(width 0)
+			(type default)
+		)
+	)
+	(wire
+		(pts
 			(xy 66.04 118.11) (xy 26.67 118.11)
 		)
@@
 	(wire
 		(pts
+			(xy 127 101.6) (xy 133.35 101.6)
+		)
+		(stroke
+			(width 0)
+			(type default)
+		)
+	)
+	(wire
+		(pts
 			(xy 276.86 36.83) (xy 279.4 36.83)
 		)
@@
 	(wire
 		(pts
+			(xy 104.14 101.6) (xy 104.14 104.14)
+		)
+		(stroke
+			(width 0)
+			(type default)
+		)
+	)
+	(wire
+		(pts
 			(xy 151.13 31.75) (xy 152.4 31.75)
 		)
@@
 	(wire
 		(pts
+			(xy 129.54 92.71) (xy 143.51 92.71)
+		)
+		(stroke
+			(width 0)
+			(type default)
+		)
+	)
+	(wire
+		(pts
 			(xy 95.25 104.14) (xy 96.52 104.14)
 		)
@@
 	(wire
 		(pts
-			(xy 354.33 27.94) (xy 359.41 27.94)
+			(xy 127 104.14) (xy 129.54 104.14)
 		)
 		(stroke
@@
 	(wire
 		(pts
-			(xy 96.52 92.71) (xy 143.51 92.71)
+			(xy 354.33 27.94) (xy 359.41 27.94)
 		)
 		(stroke
@@
 	(wire
 		(pts
+			(xy 133.35 101.6) (xy 133.35 99.06)
+		)
+		(stroke
+			(width 0)
+			(type default)
+		)
+	)
+	(wire
+		(pts
 			(xy 161.29 143.51) (xy 163.83 143.51)
 		)
@@
 	)
 	(symbol
-		(lib_id "AP63203WU-7:AP63203WU-7")
-		(at 96.52 99.06 0)
-		(unit 1)
-		(exclude_from_sim no)
-		(in_bom yes)
-		(on_board yes)
-		(dnp no)
-		(fields_autoplaced yes)
-		(property "Reference" "U4"
-			(at 116.84 88.9 0)
-			(effects
-				(font
-					(size 1.524 1.524)
-				)
-			)
-		)
-		(property "Value" "AP63203WU-7"
-			(at 116.84 91.44 0)
-			(effects
-				(font
-					(size 1.524 1.524)
-				)
-			)
-		)
-		(property "Footprint" "AP63203WU-7_DIO"
-			(at 96.52 99.06 0)
-			(effects
-				(font
-					(size 1.27 1.27)
-					(italic yes)
-				)
-				(hide yes)
-			)
-		)
-		(property "Datasheet" "AP63203WU-7"
-			(at 96.52 99.06 0)
-			(effects
-				(font
-					(size 1.27 1.27)
-					(italic yes)
-				)
-				(hide yes)
-			)
-		)
-		(property "Description" ""
-			(at 96.52 99.06 0)
-			(effects
-				(font
-					(size 1.27 1.27)
-				)
-				(hide yes)
-			)
-		)
-		(pin "1"
-		)
-		(pin "6"
-		)
-		(pin "3"
-		)
-		(pin "5"
-		)
-		(pin "4"
-		)
-		(pin "2"
-		)
-		(instances
-			(project "project"
-				(path "/f99403a2-5f0d-4f36-8249-ee7d0699b27a"
-					(reference "U4")
-					(unit 1)
-				)
-			)
-		)
-	)
-	(symbol
 		(lib_id "power:GND")
 		(at 118.11 69.85 0)
@@
 					(unit 1)
 				)
+			)
+		)
+	)
+	(symbol
+		(lib_id "Regulator_Switching:AP63203WU")
+		(at 116.84 101.6 0)
+		(unit 1)
+		(exclude_from_sim no)
+		(in_bom yes)
+		(on_board yes)
+		(dnp no)
+		(fields_autoplaced yes)
+		(property "Reference" "U4"
+			(at 116.84 91.44 0)
+			(effects
+				(font
+					(size 1.27 1.27)
+				)
+			)
+		)
+		(property "Value" "AP63203WU"
+			(at 116.84 93.98 0)
+			(effects
+				(font
+					(size 1.27 1.27)
+				)
+			)
+		)
+		(property "Footprint" "Package_TO_SOT_SMD:TSOT-23-6"
+			(at 116.84 124.46 0)
+			(effects
+				(font
+					(size 1.27 1.27)
+				)
+				(hide yes)
+			)
+		)
+		(property "Datasheet" "https://www.diodes.com/assets/Datasheets/AP63200-AP63201-AP63203-AP63205.pdf"
+			(at 116.84 101.6 0)
+			(effects
+				(font
+					(size 1.27 1.27)
+				)
+				(hide yes)
+			)
+		)
+		(property "Description" "2A, 1.1MHz Buck DC/DC Converter, fixed 3.3V output voltage, TSOT-23-6"
+			(at 116.84 101.6 0)
+			(effects
+				(font
+					(size 1.27 1.27)
+				)
+				(hide yes)
+			)
+		)
+		(pin "1"
+		)
+		(pin "3"
+		)
+		(pin "2"
+		)
+		(pin "4"
+		)
+		(pin "5"
+		)
+		(pin "6"
+		)
+		(instances
+			(project ""
+				(path "/f99403a2-5f0d-4f36-8249-ee7d0699b27a"
+					(reference "U4")
+					(unit 1)
+				)

Commit message: Footprints updated
Parts:
- U1, U3: footprint DRV8833PWPR:IC_DRV8833PWPR -> Footprint:DRV8833PWPR
- U10, U9: footprint TPS22965DSGR:SON50P200X200X80-9N -> Footprint:TPS22965DSGR
- U5: footprint TP4056:SOP127P600X175-9N -> Footprint:TP4056
- U8: footprint INA219AIDCNR:SOT65P280X145-8N -> Footprint:INA219AIDCNR
Changed lines of the file:
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@@
 			)
 		)
-		(property "Footprint" "TPS22965DSGR:SON50P200X200X80-9N"
+		(property "Footprint" "Footprint:TPS22965DSGR"
 			(at 119.38 147.32 0)
 			(effects
@@
 			)
 		)
-		(property "Footprint" "TP4056:SOP127P600X175-9N"
+		(property "Footprint" "Footprint:TP4056"
 			(at 179.07 104.14 0)
 			(effects
@@
 			)
 		)
-		(property "Footprint" "TPS22965DSGR:SON50P200X200X80-9N"
+		(property "Footprint" "Footprint:TPS22965DSGR"
 			(at 182.88 143.51 0)
 			(effects
@@
 			)
 		)
-		(property "Footprint" "DRV8833PWPR:IC_DRV8833PWPR"
+		(property "Footprint" "Footprint:DRV8833PWPR"
 			(at 172.72 46.99 0)
 			(effects
@@
 			)
 		)
-		(property "Footprint" "DRV8833PWPR:IC_DRV8833PWPR"
+		(property "Footprint" "Footprint:DRV8833PWPR"
 			(at 97.79 46.99 0)
 			(effects
@@
 			)
 		)
-		(property "Footprint" "INA219AIDCNR:SOT65P280X145-8N"
+		(property "Footprint" "Footprint:INA219AIDCNR"
 			(at 46.99 101.6 0)
 			(effects

Commit message: footprint assignment
Parts:
- removed BATTER+1: TestPoint, symbol Connector:TestPoint
- removed D1, D2: LED, LED_SMD:LED_0402_1005Metric_Pad0.77x0.64mm_HandSolder, symbol Device:LED
- removed TP4: TestPoint, TestPoint:TestPoint_Pad_D2.0mm, symbol Connector:TestPoint
- added R15: 1.5K, Resistor_SMD:R_0402_1005Metric_Pad0.72x0.64mm_HandSolder, symbol Device:R_Small
- added R16: 3m, symbol Device:R_Shunt
- added TP15, TP16, TP4: TestPoint_2Pole, symbol Connector:TestPoint_2Pole
- added U11: TS5A3159ADBVR, Package_TO_SOT_SMD:SOT-23-6, symbol Analog_Switch:TS5A3159ADBVR
- C1, C16, C17: LCSC (none) -> C52923
- C10: value C_Small -> 47u; footprint Capacitor_SMD:C_0402_1005Metric_Pad0.74x0.62mm_HandSolder -> Capacitor_SMD:C_0805_2012Metric_Pad1.18x1.45mm_HandSolder; LCSC (none) -> C16780
- C11: value C_Small -> 10u; LCSC (none) -> C15525
- C12, C8: value 0.01uF -> 10nF; LCSC (none) -> C15525
- C13, C6: LCSC (none) -> C23733
- C14, C15: footprint Capacitor_SMD:C_0402_1005Metric_Pad0.74x0.62mm_HandSolder -> Capacitor_SMD:C_0603_1608Metric_Pad1.08x0.95mm_HandSolder; LCSC (none) -> C59461
- C2, C4, C7: LCSC (none) -> C15525
- C3, C5: LCSC (none) -> C12530
- C9: value C_Small -> 100n; LCSC (none) -> C1525
- J2: footprint (none) -> Library:CONN_TYPE-C-6P_SHN
- L1: footprint Inductor_SMD:L_0402_1005Metric_Pad0.77x0.64mm_HandSolder -> Inductor_SMD:L_0805_2012Metric_Pad1.05x1.20mm_HandSolder; LCSC (none) -> C74314
- L2: footprint (none) -> Inductor_SMD:L_0805_2012Metric_Pad1.05x1.20mm_HandSolder; LCSC (none) -> C74314
- R1, R12, R13: LCSC (none) -> C11702
- R10: value 57K -> 51K; LCSC (none) -> C25794
- R11: value 1.2k -> 5.6K
- R14, R2, R3, R5: LCSC (none) -> C25744
- R4: value 37.5K -> 33K; LCSC (none) -> C25779
- R6: value 110K -> 100K; LCSC (none) -> C25741
- R7: value 15K -> 10K; LCSC (none) -> C25744
- R8, R9: LCSC (none) -> C25900
- U4: LCSC (none) -> C780769
- U5: LCSC (none) -> C16581
Connections:
- net 9V is gone; now on net HV: C7.1, U4.2 (EN), U4.3 (IN)
- net 3V3 Out: now also U11.2
- net BATT: now also R16.1, TP4.1; no longer C11.1
- net Battery: now also C12.1, C2.2, C4.2, C8.1, U1.1 (NSLEEP), U1.12 (VM), U3.1 (NSLEEP), U3.12 (VM), U6.1 (EN), U7.4 (EN), R16.4
- net FAST_CHARGE_CTRL: now also U11.6
- net GND: now also U11.4, U11.5; no longer R11.2, U8.2 (IN-)
- net at R11.1, U5.2 (PROG): now also R15.1
- net at C10.1, L1.2, TP5.1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: now also TP15.1, TP16.1
- net at R12.1: now also TP16.2
- net at R13.1: now also TP15.2
- removed net BATTERY: C12.1, C2.2, C4.2, C8.1, U1.1 (NSLEEP), U1.12 (VM), U3.1 (NSLEEP), U3.12 (VM), U8.1 (IN+)
- new net: R15.2, U11.1
- new net: R11.2, U11.3
- new net: C11.1, TP4.2
- new net: R16.2, U8.1 (IN+)
- new net: R16.3, U8.2 (IN-)
Other:
- moved on the sheet: C10, C11, C16, C17, C7, C9, J3, L1, R11, R12, R13, R14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

Commit message: routing
Parts:
- removed TP15, TP16, TP3, TP4: TestPoint_2Pole, symbol Connector:TestPoint_2Pole
- added JP1, JP3, JP4: Jumper_2_Open, Jumper:SolderJumper-2_P1.3mm_Open_RoundedPad1.0x1.5mm, symbol Jumper:Jumper_2_Open
- added JP2: Jumper_2_Open, symbol Jumper:Jumper_2_Open
- D3: footprint (none) -> Diode_SMD:D_0402_1005Metric_Pad0.77x0.64mm_HandSolder; LCSC (none) -> C2286
- J1: footprint (none) -> Connector_PinHeader_2.54mm:PinHeader_2x16_P2.54mm_Vertical
- J3: footprint (none) -> Connector_PinHeader_2.00mm:PinHeader_1x02_P2.00mm_Vertical
- R16: value 3m -> 1m; footprint (none) -> Resistor_SMD:R_0402_1005Metric_Pad0.72x0.64mm_HandSolder; LCSC (none) -> C500635
- TP2: footprint (none) -> TestPoint:TestPoint_Pad_D2.0mm
Connections:
- net BATT: now also JP1.1 (A)
- net at U2.5 (DM): now also JP4.2 (B)
- net at U2.4 (DP): now also JP4.1 (A)
- net at C10.1, L1.2, TP5.1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: now also JP2.2 (B), JP3.1 (A)
- net at R13.1: now also JP3.2 (B)
- net at R12.1: now also JP2.1 (A)
- net at C11.1: now also JP1.2 (B)
- no-connect marks 7 -> 8

Commit message: Routing
Parts:
- J2: footprint Library:CONN_TYPE-C-6P_SHN -> Connector_USB:USB_C_Receptacle_GCT_USB4135-GF-A_6P_TopMnt_Horizontal
- JP2: footprint (none) -> Jumper:SolderJumper-2_P1.3mm_Open_RoundedPad1.0x1.5mm
- R16: value 1m -> 0.5m; footprint Resistor_SMD:R_0402_1005Metric_Pad0.72x0.64mm_HandSolder -> Resistor_THT:R_Axial_Shunt_L22.2mm_W8.0mm_PS14.30mm_P25.40mm; LCSC C500635 -> C105052
Connections:
- net GND: now also J2.S1 (SHIELD)
Changed lines of the file:
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@@
 			)
 		)
-		(property "Footprint" "Library:CONN_TYPE-C-6P_SHN"
+		(property "Footprint" "Connector_USB:USB_C_Receptacle_GCT_USB4135-GF-A_6P_TopMnt_Horizontal"
 			(at 354.33 73.66 0)
 			(effects
@@
 			)
 		)
-		(property "Footprint" ""
+		(property "Footprint" "Jumper:SolderJumper-2_P1.3mm_Open_RoundedPad1.0x1.5mm"
 			(at 179.07 85.09 0)
 			(effects
@@
 	)
 	(symbol
+		(lib_id "power:GND")
+		(at 342.9 93.98 0)
+		(unit 1)
+		(exclude_from_sim no)
+		(in_bom yes)
+		(on_board yes)
+		(dnp no)
+		(fields_autoplaced yes)
+		(property "Reference" "#PWR035"
+			(at 342.9 100.33 0)
+			(effects
+				(font
+					(size 1.27 1.27)
+				)
+				(hide yes)
+			)
+		)
+		(property "Value" "GND"
+			(at 342.9 99.06 0)
+			(effects
+				(font
+					(size 1.27 1.27)
+				)
+			)
+		)
+		(property "Footprint" ""
+			(at 342.9 93.98 0)
+			(effects
+				(font
+					(size 1.27 1.27)
+				)
+				(hide yes)
+			)
+		)
+		(property "Datasheet" ""
+			(at 342.9 93.98 0)
+			(effects
+				(font
+					(size 1.27 1.27)
+				)
+				(hide yes)
+			)
+		)
+		(property "Description" "Power symbol creates a global label with name \"GND\" , ground"
+			(at 342.9 93.98 0)
+			(effects
+				(font
+					(size 1.27 1.27)
+				)
+				(hide yes)
+			)
+		)
+		(pin "1"
+		)
+		(instances
+			(project "project"
+				(path "/f99403a2-5f0d-4f36-8249-ee7d0699b27a"
+					(reference "#PWR035")
+					(unit 1)
+				)
+			)
+		)
+	)
+	(symbol
 		(lib_id "Connector:TestPoint")
 		(at 194.31 52.07 180)
@@
 			)
 		)
-		(property "Value" "1m"
+		(property "Value" "0.5m"
 			(at 243.84 166.3699 0)
 			(effects
@@
 			)
 		)
-		(property "Footprint" "Resistor_SMD:R_0402_1005Metric_Pad0.72x0.64mm_HandSolder"
+		(property "Footprint" "Resistor_THT:R_Axial_Shunt_L22.2mm_W8.0mm_PS14.30mm_P25.40mm"
 			(at 244.602 165.1 90)
 			(effects
@@
 			)
 		)
-		(property "LCSC" "C500635"
+		(property "LCSC" "C105052"
 			(at 246.38 165.1 0)
 			(effects

Commit message: checks
Parts:
- R16: footprint Resistor_THT:R_Axial_Shunt_L22.2mm_W8.0mm_PS14.30mm_P25.40mm -> Resistor_SMD:R_Shunt_Vishay_WSR2_WSR3; LCSC C105052 -> C252656
Connections:
- net 3V3 is gone; now on net 3V3 Out: R8.1, R9.1, U8.4 (VS), U8.7 (A0)
Changed lines of the file:
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@@
 	(rectangle
 		(start 77.47 167.64)
-		(end 208.28 208.28)
+		(end 219.71 208.28)
 		(stroke
 			(width 0)
@@
 		)
 	)
-	(label "3V3"
-		(at 316.23 153.67 0)
-		(effects
-			(font
-				(size 1.27 1.27)
-			)
-			(justify left bottom)
-		)
-	)
 	(label "MOTOR3_B_OUT"
 		(at 123.19 44.45 0)
@@
 	)
 	(label "EXT_LOAD1_OUT"
-		(at 204.47 184.15 90)
+		(at 204.47 184.15 0)
 		(effects
 			(font
@@
 		)
 	)
+	(label "3V3 Out"
+		(at 316.23 153.67 0)
+		(effects
+			(font
+				(size 1.27 1.27)
+			)
+			(justify left bottom)
+		)
+	)
 	(label "5V Out"
 		(at 383.54 146.05 0)
@@
 		(dnp no)
 		(property "Reference" "TP14"
-			(at 138.43 181.61 0)
+			(at 134.112 180.848 0)
 			(effects
 				(font
@@
 		)
 		(property "Value" "TestPoint"
-			(at 138.43 183.388 0)
+			(at 132.842 182.626 0)
 			(effects
 				(font
@@
 		(on_board yes)
 		(dnp no)
-		(fields_autoplaced yes)
 		(property "Reference" "TP1"
-			(at 204.47 179.5779 0)
+			(at 200.152 177.038 0)
 			(effects
 				(font
@@
 		)
 		(property "Value" "TestPoint"
-			(at 204.47 182.1179 0)
+			(at 199.136 179.07 0)
 			(effects
 				(font
@@
 			)
 		)
-		(property "Footprint" "Resistor_THT:R_Axial_Shunt_L22.2mm_W8.0mm_PS14.30mm_P25.40mm"
+		(property "Footprint" "Resistor_SMD:R_Shunt_Vishay_WSR2_WSR3"
 			(at 244.602 165.1 90)
 			(effects
@@
 			)
 		)
-		(property "LCSC" "C105052"
+		(property "LCSC" "C252656"
 			(at 246.38 165.1 0)
 			(effects
