File: project/_autosave-project.kicad_sch (KiCad schematic)
At the start: 67 parts, among them J1 Conn_02x16_Odd_Even, J2 TYPE-C 6P(040新), J3 Conn_01x02_Pin, SW1 SS-12D10L9, U1 DRV8833PWPR, U10 TPS22965DSGR, U11 TS5A3159ADBVR, U2 CH224K, U3 DRV8833PWPR, U4 AP63203WU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

Commit message: Updates
Changes datasheet names,updates PCB,fixex errors
Parts:
- J3: footprint Connector_PinHeader_2.00mm:PinHeader_1x02_P2.00mm_Vertical -> Connector_JST:JST_PH_B2B-PH-K_1x02_P2.00mm_Vertical
Changed lines of the file:
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@@
 			)
 		)
-		(property "Footprint" "Connector_PinHeader_2.00mm:PinHeader_1x02_P2.00mm_Vertical"
+		(property "Footprint" "Connector_JST:JST_PH_B2B-PH-K_1x02_P2.00mm_Vertical"
 			(at 113.03 82.55 0)
 			(effects
