File: project/_autosave-project.kicad_pcb (KiCad board)
At the start: 2 copper layers, 80 x 60 mm, 69 parts, among them J1 Conn_02x16_Odd_Even, J2 TYPE-C 6P(040新), J3 Conn_01x02_Pin, SW1 SS-12D10L9, U1 DRV8833PWPR, U10 TPS22965DSGR, U11 TS5A3159ADBVR, U2 CH224K, U3 DRV8833PWPR, U4 AP63203WU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

Commit message: assigning correct footprints
Parts:
- moved C16 3.69 mm to (139.0, 80.1)
- moved R8 3.69 mm to (139.5, 76.3)
- moved R9 3.69 mm to (143.5, 77.3)
- moved U8 3.69 mm to (148.2, 76.5)
Other:
- board text added: "TMBTLA001 MDLOXO001 GROUP 65"
Changed lines of the file:
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@@
 	(footprint "Resistor_SMD:R_0402_1005Metric_Pad0.72x0.64mm_HandSolder"
 		(layer "F.Cu")
-		(at 146 74.5525 90)
+		(at 143.49 77.2525 90)
 		(descr "Resistor SMD 0402 (1005 Metric), square (rectangular) end terminal, IPC_7351 nominal with elongated pad for handsoldering. (Body size source: IPC-SM-782 page 72, https://www.pcb-3d.com/wordpress/wp-content/uploads/ipc-sm-782a_amendment_1_and_2.pdf), generated with kicad-footprint-generator")
 		(tags "resistor handsolder")
@@
 	(footprint "Capacitor_SMD:C_0402_1005Metric_Pad0.74x0.62mm_HandSolder"
 		(layer "F.Cu")
-		(at 141.5 77.3875 90)
+		(at 138.99 80.0875 90)
 		(descr "Capacitor SMD 0402 (1005 Metric), square (rectangular) end terminal, IPC_7351 nominal with elongated pad for handsoldering. (Body size source: IPC-SM-782 page 76, https://www.pcb-3d.com/wordpress/wp-content/uploads/ipc-sm-782a_amendment_1_and_2.pdf), generated with kicad-footprint-generator")
 		(tags "capacitor handsolder")
@@
 	(footprint "Resistor_SMD:R_0402_1005Metric_Pad0.72x0.64mm_HandSolder"
 		(layer "F.Cu")
-		(at 142 73.5525 90)
+		(at 139.49 76.2525 90)
 		(descr "Resistor SMD 0402 (1005 Metric), square (rectangular) end terminal, IPC_7351 nominal with elongated pad for handsoldering. (Body size source: IPC-SM-782 page 72, https://www.pcb-3d.com/wordpress/wp-content/uploads/ipc-sm-782a_amendment_1_and_2.pdf), generated with kicad-footprint-generator")
 		(tags "resistor handsolder")
@@
 	(footprint "Footprint:INA219AIDCNR"
 		(layer "F.Cu")
-		(at 150.755 73.825 180)
+		(at 148.245 76.525 180)
 		(property "Reference" "U8"
 			(at 0.925 -2.635 0)
@@
 		(layer "Edge.Cuts")
 	)
+	(gr_text "TMBTLA001\nMDLOXO001\nGROUP 65"
+		(at 119.5 109.5 0)
+		(layer "B.SilkS")
+		(effects
+			(font
+				(size 1.5 1.5)
+				(thickness 0.3)
+				(bold yes)
+			)
+			(justify left bottom)
+		)
+	)
 	(embedded_fonts no)
